File: Kicad/ECE 412.kicad_sch (KiCad schematic)
At the start: 16 parts, among them U2 3405, U3 MIC5219-3.3YMM, U4 LMC6042IM, U5 MAX1032BEUG_

Commit message: Add files via upload
Parts:
- added J1: Faraday Cup IN, Connector_PinHeader_2.54mm:PinHeader_1x01_P2.54mm_Vertical, symbol Connector:Conn_01x01_Pin
- added J2: 3.3V, Connector_PinHeader_2.54mm:PinHeader_1x02_P2.54mm_Vertical, symbol Connector:Conn_01x02_Pin
- added R6: 150k, XIAO_:R_Axial_DIN0207_L6.3mm_D2.5mm_P10.16mm_Horizontal_2.54_pad, symbol Device:R
- added R7: 470k, XIAO_:R_Axial_DIN0207_L6.3mm_D2.5mm_P10.16mm_Horizontal_2.54_pad, symbol Device:R
- added TP1, TP2, TP3, TP4: TestPoint, TestPoint:TestPoint_THTPad_D2.0mm_Drill1.0mm, symbol Connector:TestPoint
- C1, C3, C4: footprint (none) -> Capacitor_THT:CP_Radial_D5.0mm_P2.00mm
- C2: footprint (none) -> Capacitor_THT:CP_Radial_Tantal_D5.0mm_P5.00mm
- C5: value 500p -> 100p; footprint (none) -> Capacitor_THT:CP_Radial_Tantal_D5.0mm_P5.00mm
- R1, R2, R4: value 1K -> 10k; footprint (none) -> XIAO_:R_Axial_DIN0207_L6.3mm_D2.5mm_P10.16mm_Horizontal_2.54_pad
- R3: footprint (none) -> XIAO_:R_Vishay_TR10X5G00JNES
- R5: value 100K -> 40k; footprint (none) -> XIAO_:R_Axial_DIN0207_L6.3mm_D2.5mm_P10.16mm_Horizontal_2.54_pad
- U2: footprint MODULE_3405 -> 3405_Huzzah:MODULE_3405
- U4: value LMC6042IM -> LMC662; footprint SOIC127P599X175-8N -> LMC662AIMX_NOPB:SOIC127P599X175-8N
- U5: footprint SOP65P640X110-24N -> MAX1032BEUGT:SOP65P640X110-24N
- Vbat1: renamed from Vbat; footprint (none) -> Connector_PinHeader_2.54mm:PinHeader_1x02_P2.54mm_Vertical
Connections:
- net 4.5V: now also TP1.1
- net Faraday Cup: now also J1.1 (Pin_1)
- net GND: now also U5.24 (AGND1), J2.2 (Pin_2)
- net at C3.1, R1.1, U4.8 (V+)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: no longer U3.1 (EN), U3.2 (IN)
- net 3.3V: now reaches DS1.28 (VCC), U2.15 (3V), U5.1 (AVDD1), U5.20 (REF)
- net 3.3V: now also J2.1 (Pin_1); no longer C1.1, C2.1, U3.3 (OUT), U5.18 (DVDD)
- net at C5.1, R3.1, R4.2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: now also TP2.1
- net at R4.1, R5.2, U4.6 (NEGB): now also R6.2, R7.2
- net at R5.1, U4.7 (OUTB), U5.2 (CH0): now also R6.1, R7.1, TP3.1
- net at U2.4 (MISO/IO19), U5.14 (DOUT): now also TP4.1
- new net: U3.1 (EN), U3.2 (IN)
- new net: C1.1, C2.1, U3.3 (OUT)
Other:
- note removed: "#2"
- note removed: "02/16/2025"
- note removed: "1"
- note removed: "Rough Draft Schematic"
- note removed: "TEAM 3 - COATL-AIRCRAFT"
- company: (none) -> Annika Boyd, Eisa Alsharifi, Felix Moss, Nathan Truong
- title: (none) -> Team 3 - COATL Aircraft Schematic
- moved on the sheet: C5, R1, R2, R3, R4, R5, U4

Commit message: Add files via upload
Parts:
- removed J2: 3.3V, Connector_PinHeader_2.54mm:PinHeader_1x02_P2.54mm_Vertical, symbol Connector:Conn_01x02_Pin
- removed U2: 3405, 3405_Huzzah:MODULE_3405, symbol 3405:3405
- removed U3: MIC5219-3.3YMM, Package_SO:MSOP-8_3x3mm_P0.65mm, symbol Regulator_Linear:MIC5219-3.3YMM
- added A1: Adafruit_Feather_HUZZAH32_ESP32, Module:Adafruit_Feather, symbol MCU_Module:Adafruit_Feather_HUZZAH32_ESP32
- added TP10: ADC DIN, TestPoint:TestPoint_THTPad_D2.0mm_Drill1.0mm, symbol Connector:TestPoint
- added TP11: ADC CS, TestPoint:TestPoint_THTPad_D2.0mm_Drill1.0mm, symbol Connector:TestPoint
- added TP4: Vout2, TestPoint:TestPoint_THTPad_D2.0mm_Drill1.0mm, symbol Connector:TestPoint
- added TP5: 470k switch, TestPoint:TestPoint_THTPad_D2.0mm_Drill1.0mm, symbol Connector:TestPoint
- added TP6: 150k switch, TestPoint:TestPoint_THTPad_D2.0mm_Drill1.0mm, symbol Connector:TestPoint
- added TP7: 40k switch, TestPoint:TestPoint_THTPad_D2.0mm_Drill1.0mm, symbol Connector:TestPoint
- added TP8: ADC Vref, TestPoint:TestPoint_THTPad_D2.0mm_Drill1.0mm, symbol Connector:TestPoint
- added TP9: ADC SCLK, TestPoint:TestPoint_THTPad_D2.0mm_Drill1.0mm, symbol Connector:TestPoint
- added U1: LM7805_TO220, Package_TO_SOT_THT:TO-220-3_Vertical, symbol Regulator_Linear:LM7805_TO220
- added U2: ADG441BN, ADG441BN:DIP254P762X533-16P, symbol ADG441BN:ADG441BN
- C1: footprint Capacitor_THT:CP_Radial_D5.0mm_P2.00mm -> Capacitor_THT:C_Radial_D6.3mm_H5.0mm_P2.50mm
- C2: footprint Capacitor_THT:CP_Radial_Tantal_D5.0mm_P5.00mm -> Capacitor_THT:C_Radial_D6.3mm_H5.0mm_P2.50mm
- C3: value 10uF -> 0.1uF; footprint Capacitor_THT:CP_Radial_D5.0mm_P2.00mm -> Capacitor_THT:C_Radial_D6.3mm_H5.0mm_P2.50mm
- C4: value 10uF -> 1uF; footprint Capacitor_THT:CP_Radial_D5.0mm_P2.00mm -> Capacitor_THT:C_Radial_D6.3mm_H5.0mm_P2.50mm
- C5: footprint Capacitor_THT:CP_Radial_Tantal_D5.0mm_P5.00mm -> Capacitor_THT:C_Radial_D10.0mm_H12.5mm_P5.00mm
- TP1: value TestPoint -> 4.5V
- TP12: renamed from TP4; value TestPoint -> ADC Dout
- TP2: value TestPoint -> 5V
- TP3: value TestPoint -> Vout1
- U4: footprint LMC662AIMX_NOPB:SOIC127P599X175-8N -> Package_DIP:DIP-8_W7.62mm
Connections:
- net 3.3V: now also U5.17 (DVDD0), U5.18 (DVDD), A1.2 (3V3); no longer DS1.28 (VCC), U5.1 (AVDD1), U5.20 (REF)
- net GND: now also C3.1, U5.15 (DGND0), U5.16 (DGND), U5.21 (AGND3), U5.23 (AGND2), U5.3 (CH1), U5.4 (CH2), U5.5 (CH3), A1.4 (GND), U1.2 (GND), U2.4 (VSS), U2.5 (GND), U2.8 (IN4); no longer C3.2, DS1.1 (GND), DS1.16 (R/~{W}), DS1.17 (E/~{RD}), DS1.30 (GND)
- net at C5.1, R3.1, R4.2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: now also TP3.1; no longer TP2.1
- net 5V: now reaches C1.1, C2.1
- net 5V: now also TP2.1, U5.1 (AVDD1), U5.22 (AVDD2), A1.28 (VBAT), U1.3 (VO)
- net 9V: now reaches R1.1, U4.8 (V+), Vbat1.1 (+)
- net 9V: now also U1.1 (VI), U2.13 (VDD); no longer C3.1
- net at U5.10 (~{CS}): now also A1.7 (I34/A2), TP11.1
- net at TP12.1, U5.14 (DOUT): now also A1.13 (MISO/IO19)
- net at DS1.23 (D5): no longer U5.11 (DIN)
- net at DS1.22 (D4): no longer U5.13 (SCLK)
- net at C4.1, U5.19 (REFCAP): now also TP8.1
- net Faraday Cup renamed Charge IN
- new net: A1.19 (A6/IO14), TP7.1, U2.9 (IN3)
- new net: A1.22 (A9/IO33), TP5.1, U2.1 (IN1)
- new net: R5.1, U2.10 (D3)
- new net: TP4.1, U2.11 (S3), U2.14 (S2), U2.3 (S1), U4.7 (OUTB), U5.2 (CH0)
- new net: R6.1, U2.15 (D2)
- new net: A1.20 (A7/IO32), TP6.1, U2.16 (IN2)
- new net: R7.1, U2.2 (D1)
- new net: DS1.1 (GND), DS1.30 (GND)
- new net: A1.12 (MOSI/IO18), TP10.1, U5.11 (DIN)
- new net: A1.11 (SCK/IO5), TP9.1, U5.13 (SCLK)
- new net: C3.2, U5.20 (REF)
- no-connect marks 53 -> 22
Other:
- note added: "Analog GND"
- note added: "Analog Switches"
- note added: "CS(PIN 10) -> IO34"
- note added: "Digital GND"
- note added: "Voltage Regulator 5V Output"
- note removed: "3.3V"
- note removed: "CS(PIN 10) -> IO21"
- moved on the sheet: C1, C2, C4, C5, DS1, J1, R1, R2, R3, R4, R5, R6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

Commit message: Add files via upload
Parts:
- removed U2: ADG441BN, ADG441BN:DIP254P762X533-16P, symbol ADG441BN:ADG441BN
- added C10, C11, C13, C14, C15, C17, C19, C7, C8: 0.1uF, Capacitor_SMD:C_0805_2012Metric_Pad1.18x1.45mm_HandSolder, symbol Device:C
- added C12: 100pF, Capacitor_SMD:C_0805_2012Metric_Pad1.18x1.45mm_HandSolder, symbol Device:C
- added C16, C18, C6: 10uF, Capacitor_SMD:C_0805_2012Metric_Pad1.18x1.45mm_HandSolder, symbol Device:C
- added C9: 1uF, Capacitor_SMD:C_0805_2012Metric_Pad1.18x1.45mm_HandSolder, symbol Device:C
- added IC1: ADG412, ADG412:TSSOP16, symbol ADG412:ADG412
- C1, C2, C4: footprint Capacitor_THT:C_Radial_D6.3mm_H5.0mm_P2.50mm -> Capacitor_SMD:C_0805_2012Metric_Pad1.18x1.45mm_HandSolder
- C3: value 0.1uF -> 1uF; footprint Capacitor_THT:C_Radial_D6.3mm_H5.0mm_P2.50mm -> Capacitor_SMD:C_0805_2012Metric_Pad1.18x1.45mm_HandSolder
Connections:
- net 3.3V: now also C11.2, C8.2, C9.1
- net 4.5V: now also C18.1, C19.1
- net 5V: now also C10.1, C6.1, C7.1, IC1.12 (VL)
- net 9V: now also C16.1, C17.1, IC1.13 (VDD)
- net GND: now also C10.2, C11.1, C12.1, C13.1, C14.1, C15.1, C16.2, C17.2, C18.2, C19.2, C6.2, C7.2, C8.1, C9.2, IC1.4 (VSS), IC1.5 (GND), IC1.8; no longer U5.3 (CH1), U5.4 (CH2), U5.5 (CH3)
- net at A1.19 (A6/IO14), TP7.1: now also IC1.9
- net at A1.22 (A9/IO33), TP5.1: now also IC1.1
- net at R5.1: now also IC1.10
- net at TP4.1, U4.7 (OUTB), U5.2 (CH0): now also C12.2, IC1.11, IC1.14, IC1.3
- net at R6.1: now also IC1.15
- net at A1.20 (A7/IO32), TP6.1: now also IC1.16
- net at R7.1: now also IC1.2
- new net: C14.2, U5.4 (CH2)
- new net: C13.2, U5.3 (CH1)
- new net: C15.2, U5.5 (CH3)
Other:
- moved on the sheet: R5, R6, R7, TP12, TP5, TP6, TP7

Commit message: Add files via upload
Parts:
- IC1: footprint ADG412:TSSOP16 -> ADG412:SOIC16N
Changed lines of the file:
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@@
 			)
 		)
-		(property "Footprint" "ADG412:TSSOP16"
+		(property "Footprint" "ADG412:SOIC16N"
 			(at 160.02 110.49 0)
 			(effects
@@
 			)
 		)
-		(property "Footprint" "ADG412:TSSOP16"
+		(property "Footprint" "ADG412:SOIC16N"
 			(at 160.02 85.09 0)
 			(effects
@@
 			)
 		)
-		(property "Footprint" "ADG412:TSSOP16"
+		(property "Footprint" "ADG412:SOIC16N"
 			(at 160.02 97.79 0)
 			(effects
@@
 			)
 		)
-		(property "Footprint" "ADG412:TSSOP16"
+		(property "Footprint" "ADG412:SOIC16N"
 			(at 160.02 123.19 0)
 			(effects
@@
 			)
 		)
-		(property "Footprint" "ADG412:TSSOP16"
+		(property "Footprint" "ADG412:SOIC16N"
 			(at 161.29 69.85 0)
 			(effects

Commit message: Add files via upload
Parts:
- C1: value 10uF -> 1uF; footprint Capacitor_SMD:C_0805_2012Metric_Pad1.18x1.45mm_HandSolder -> Capacitor_SMD:C_1206_3216Metric_Pad1.33x1.80mm_HandSolder
- C10, C11, C12, C13, C14, C15, C16, C17, C18, C19, C2, C3, C4, C6, C7, C8, C9: footprint Capacitor_SMD:C_0805_2012Metric_Pad1.18x1.45mm_HandSolder -> Capacitor_SMD:C_1206_3216Metric_Pad1.33x1.80mm_HandSolder
- R1, R2, R4, R5, R6, R7: footprint XIAO_:R_Axial_DIN0207_L6.3mm_D2.5mm_P10.16mm_Horizontal_2.54_pad -> Resistor_SMD:R_0805_2012Metric_Pad1.20x1.40mm_HandSolder
Connections:
- no-connect marks 22 -> 23
Changed lines of the file:
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@@
 	)
 	(no_connect
+		(at 261.62 105.41)
+	)
+	(no_connect
 		(at 269.24 123.19)
 	)
@@
 			)
 		)
-		(property "Footprint" "Capacitor_SMD:C_0805_2012Metric_Pad1.18x1.45mm_HandSolder"
+		(property "Footprint" "Capacitor_SMD:C_1206_3216Metric_Pad1.33x1.80mm_HandSolder"
 			(at 91.7448 229.87 0)
 			(effects
@@
 			)
 		)
-		(property "Footprint" "Capacitor_SMD:C_0805_2012Metric_Pad1.18x1.45mm_HandSolder"
+		(property "Footprint" "Capacitor_SMD:C_1206_3216Metric_Pad1.33x1.80mm_HandSolder"
 			(at 73.3552 50.8 0)
 			(effects
@@
 			)
 		)
-		(property "Footprint" "Capacitor_SMD:C_0805_2012Metric_Pad1.18x1.45mm_HandSolder"
+		(property "Footprint" "Capacitor_SMD:C_1206_3216Metric_Pad1.33x1.80mm_HandSolder"
 			(at 84.7852 31.75 0)
 			(effects
@@
 			)
 		)
-		(property "Footprint" "XIAO_:R_Axial_DIN0207_L6.3mm_D2.5mm_P10.16mm_Horizontal_2.54_pad"
+		(property "Footprint" "Resistor_SMD:R_0805_2012Metric_Pad1.20x1.40mm_HandSolder"
 			(at 114.3 83.312 90)
 			(effects
@@
 			)
 		)
-		(property "Footprint" "Capacitor_SMD:C_0805_2012Metric_Pad1.18x1.45mm_HandSolder"
+		(property "Footprint" "Capacitor_SMD:C_1206_3216Metric_Pad1.33x1.80mm_HandSolder"
 			(at 118.4148 237.49 0)
 			(effects
@@
 			)
 		)
-		(property "Value" "10uF"
+		(property "Value" "1uF"
 			(at 168.91 29.2099 0)
 			(effects
@@
 			)
 		)
-		(property "Footprint" "Capacitor_SMD:C_0805_2012Metric_Pad1.18x1.45mm_HandSolder"
+		(property "Footprint" "Capacitor_SMD:C_1206_3216Metric_Pad1.33x1.80mm_HandSolder"
 			(at 166.0652 31.75 0)
 			(effects
@@
 			)
 		)
-		(property "Footprint" "Capacitor_SMD:C_0805_2012Metric_Pad1.18x1.45mm_HandSolder"
+		(property "Footprint" "Capacitor_SMD:C_1206_3216Metric_Pad1.33x1.80mm_HandSolder"
 			(at 110.49 216.8652 0)
 			(effects
@@
 			)
 		)
-		(property "Footprint" "Capacitor_SMD:C_0805_2012Metric_Pad1.18x1.45mm_HandSolder"
+		(property "Footprint" "Capacitor_SMD:C_1206_3216Metric_Pad1.33x1.80mm_HandSolder"
 			(at 106.9848 237.49 0)
 			(effects
@@
 			)
 		)
-		(property "Footprint" "XIAO_:R_Axial_DIN0207_L6.3mm_D2.5mm_P10.16mm_Horizontal_2.54_pad"
+		(property "Footprint" "Resistor_SMD:R_0805_2012Metric_Pad1.20x1.40mm_HandSolder"
 			(at 96.52 106.172 90)
 			(effects
@@
 			)
 		)
-		(property "Footprint" "XIAO_:R_Axial_DIN0207_L6.3mm_D2.5mm_P10.16mm_Horizontal_2.54_pad"
+		(property "Footprint" "Resistor_SMD:R_0805_2012Metric_Pad1.20x1.40mm_HandSolder"
 			(at 114.3 94.742 90)
 			(effects
@@
 			)
 		)
-		(property "Footprint" "Capacitor_SMD:C_0805_2012Metric_Pad1.18x1.45mm_HandSolder"
+		(property "Footprint" "Capacitor_SMD:C_1206_3216Metric_Pad1.33x1.80mm_HandSolder"
 			(at 129.8448 237.49 0)
 			(effects
@@
 			)
 		)
-		(property "Footprint" "XIAO_:R_Axial_DIN0207_L6.3mm_D2.5mm_P10.16mm_Horizontal_2.54_pad"
+		(property "Footprint" "Resistor_SMD:R_0805_2012Metric_Pad1.20x1.40mm_HandSolder"
 			(at 33.782 33.02 90)
 			(effects
@@
 			)
 		)
-		(property "Footprint" "XIAO_:R_Axial_DIN0207_L6.3mm_D2.5mm_P10.16mm_Horizontal_2.54_pad"
+		(property "Footprint" "Resistor_SMD:R_0805_2012Metric_Pad1.20x1.40mm_HandSolder"
 			(at 114.3 106.172 90)
 			(effects
@@
 			)
 		)
-		(property "Footprint" "Capacitor_SMD:C_0805_2012Metric_Pad1.18x1.45mm_HandSolder"
+		(property "Footprint" "Capacitor_SMD:C_1206_3216Metric_Pad1.33x1.80mm_HandSolder"
 			(at 232.41 197.1548 0)
 			(effects
@@
 			)
 		)
-		(property "Footprint" "Capacitor_SMD:C_0805_2012Metric_Pad1.18x1.45mm_HandSolder"
+		(property "Footprint" "Capacitor_SMD:C_1206_3216Metric_Pad1.33x1.80mm_HandSolder"
 			(at 232.41 185.7248 0)
 			(effects
@@
 			)
 		)
-		(property "Footprint" "XIAO_:R_Axial_DIN0207_L6.3mm_D2.5mm_P10.16mm_Horizontal_2.54_pad"
+		(property "Footprint" "Resistor_SMD:R_0805_2012Metric_Pad1.20x1.40mm_HandSolder"
 			(at 33.782 45.72 90)
 			(effects
@@
 			)
 		)
-		(property "Footprint" "Capacitor_SMD:C_0805_2012Metric_Pad1.18x1.45mm_HandSolder"
+		(property "Footprint" "Capacitor_SMD:C_1206_3216Metric_Pad1.33x1.80mm_HandSolder"
 			(at 61.9252 50.8 0)
 			(effects
@@
 			)
 		)
-		(property "Footprint" "Capacitor_SMD:C_0805_2012Metric_Pad1.18x1.45mm_HandSolder"
+		(property "Footprint" "Capacitor_SMD:C_1206_3216Metric_Pad1.33x1.80mm_HandSolder"
 			(at 231.14 232.1052 0)
 			(effects
@@
 			)
 		)
-		(property "Footprint" "Capacitor_SMD:C_0805_2012Metric_Pad1.18x1.45mm_HandSolder"
+		(property "Footprint" "Capacitor_SMD:C_1206_3216Metric_Pad1.33x1.80mm_HandSolder"
 			(at 232.41 209.8548 0)
 			(effects
@@
 			)
 		)
-		(property "Footprint" "Capacitor_SMD:C_0805_2012Metric_Pad1.18x1.45mm_HandSolder"
+		(property "Footprint" "Capacitor_SMD:C_1206_3216Metric_Pad1.33x1.80mm_HandSolder"
 			(at 223.52 239.0648 0)
 			(effects
@@
 			)
 		)
-		(property "Footprint" "Capacitor_SMD:C_0805_2012Metric_Pad1.18x1.45mm_HandSolder"
+		(property "Footprint" "Capacitor_SMD:C_1206_3216Metric_Pad1.33x1.80mm_HandSolder"
 			(at 177.4952 31.75 0)
 			(effects
@@
 			)
 		)
-		(property "Footprint" "Capacitor_SMD:C_0805_2012Metric_Pad1.18x1.45mm_HandSolder"
+		(property "Footprint" "Capacitor_SMD:C_1206_3216Metric_Pad1.33x1.80mm_HandSolder"
 			(at 118.11 203.5048 0)
 			(effects
@@
 			)
 		)
-		(property "Footprint" "Capacitor_SMD:C_0805_2012Metric_Pad1.18x1.45mm_HandSolder"
+		(property "Footprint" "Capacitor_SMD:C_1206_3216Metric_Pad1.33x1.80mm_HandSolder"
 			(at 223.52 218.7448 0)
 			(effects
@@
 			)
 		)
-		(property "Footprint" "Capacitor_SMD:C_0805_2012Metric_Pad1.18x1.45mm_HandSolder"
+		(property "Footprint" "Capacitor_SMD:C_1206_3216Metric_Pad1.33x1.80mm_HandSolder"
 			(at 73.3552 31.75 0)
 			(effects

Commit message: Add files via upload
Parts:
- removed A1: Adafruit_Feather_HUZZAH32_ESP32, Module:Adafruit_Feather, symbol MCU_Module:Adafruit_Feather_HUZZAH32_ESP32
- removed DS1: OLED-128O064D, Display:OLED-128O064D, symbol Display_Graphic:OLED-128O064D
- removed TP10: ADC DIN, TestPoint:TestPoint_THTPad_D2.0mm_Drill1.0mm, symbol Connector:TestPoint
- removed U1: LM7805_TO220, Package_TO_SOT_THT:TO-220-3_Vertical, symbol Regulator_Linear:LM7805_TO220
- removed U4: LMC662, Package_DIP:DIP-8_W7.62mm, symbol LMC6042IM:LMC6042IM
- removed U5: MAX1032BEUG_, MAX1032BEUGT:SOP65P640X110-24N, symbol MAX1032BEUG_:MAX1032BEUG_
- added C20, C21: 0.1uF, Capacitor_SMD:C_1206_3216Metric_Pad1.33x1.80mm_HandSolder, symbol Device:C
- added TP13: 40k switch, TestPoint:TestPoint_THTPad_D2.0mm_Drill1.0mm, symbol Connector:TestPoint
- added TP14: ADC Dout, TestPoint:TestPoint_THTPad_D2.0mm_Drill1.0mm, symbol Connector:TestPoint
- added U1: LMC662, Package_DIP:DIP-8_W7.62mm, symbol LMC6042IM:LMC6042IM
- added U4: MAX1032BEUG_, MAX1032BEUGT:SOP65P640X110-24N, symbol MAX1032BEUG_:MAX1032BEUG_
- added U5: BUF634AxD, Package_SO:SOIC-8_3.9x4.9mm_P1.27mm, symbol buf634axd:BUF634AxD
- added XIAO1: ~, XIAO_:XIAO_QTpy, symbol XIAO:esp32s3
- C1: value 1uF -> 100p; footprint Capacitor_SMD:C_1206_3216Metric_Pad1.33x1.80mm_HandSolder -> Capacitor_THT:C_Radial_D10.0mm_H12.5mm_P5.00mm
- C10, C11, C19: value 0.1uF -> 1uF
- C12: value 100pF -> 0.1uF
- C18, C6: value 10uF -> 0.1uF
- C2: value 0.1uF -> 10uF
- C3, C4: value 1uF -> 10uF
- C5: value 100p -> 0.1uF; footprint Capacitor_THT:C_Radial_D10.0mm_H12.5mm_P5.00mm -> Capacitor_SMD:C_1206_3216Metric_Pad1.33x1.80mm_HandSolder
- C9: value 1uF -> 100pF
- R5: value 40k -> 470k
- R7: value 470k -> 40k
- TP11: value ADC CS -> 470k switch
- TP12: value ADC Dout -> 150k switch
- TP2: value 5V -> -4.5V
- TP4: value Vout2 -> 0V
- TP5: value 470k switch -> Vout2
- TP6: value 150k switch -> ADC Vref
- TP7: value 40k switch -> ADC SCLK
- TP8: value ADC Vref -> ADC DIN
- TP9: value ADC SCLK -> ADC CS
Connections:
- net 9V is gone; now on net 4.5V: C16.1, C17.1, IC1.13 (VDD), R1.1, Vbat1.1 (+)
- net 3.3V: now also C18.2, C19.1, IC1.12 (VL), C20.2, C21.1, U4.17 (DVDD0), U4.18 (DVDD), XIAO1.3V3; no longer C11.2, C8.2, C9.1
- net 4.5V: now also C15.1, C2.1, C3.1, C5.1, C7.1, U1.8 (V+), U4.1 (AVDD1), U4.22 (AVDD2), U5.7 (V+), XIAO1.5V; no longer C18.1, C19.1, R1.2, R2.1
- net Charge IN: now also C1.2, U1.2 (NEGA); no longer C5.2
- net GND: now also C10.1, C11.2, C15.2, C18.1, C3.2, C4.1, C5.2, C8.2, C9.1, TP4.1, C20.1, C21.2, U1.3 (POSA), U1.5 (POSB), U4.12 (SSTRB), U4.15 (DGND0), U4.16 (DGND), U4.21 (AGND3), U4.23 (AGND2), U4.24 (AGND1), U5.6, XIAO1.GND; no longer C1.2, C10.2, C11.1, C15.1, C18.2, C2.2, C3.1, C4.2, C8.1, C9.2, IC1.4 (VSS), R2.2, Vbat1.2 (-)
- net at TP7.1: now also U4.13 (SCLK), XIAO1.8; no longer IC1.9
- net at IC1.11, IC1.14, IC1.3: now also C9.2, TP5.1, U1.7 (OUTB), U4.2 (CH0); no longer C12.2, TP4.1
- net at IC1.10: now also R7.1; no longer R5.1
- net at IC1.2: now also R5.1; no longer R7.1
- net at R4.1, R5.2, R6.2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: now also U1.6 (NEGB)
- net at R3.1, R4.2, TP3.1: now also C1.1, U1.1 (OUTA); no longer C5.1
- net at IC1.1: now also TP11.1, XIAO1.2; no longer TP5.1
- net at C14.2: now also U4.5 (CH3)
- net at TP12.1: now also IC1.16, XIAO1.1
- net at TP6.1: now also C11.1, U4.19 (REFCAP); no longer IC1.16
- net at TP8.1: now also U4.11 (DIN), XIAO1.10; no longer C4.1
- net at TP9.1: now also U4.10 (~{CS}), XIAO1.3
- net at C13.2: now also U4.4 (CH2)
- removed net 5V: C1.1, C10.1, C2.1, C6.1, C7.1, IC1.12 (VL), TP2.1
- new net: R1.2, R2.1, U5.3 (V_{IN})
- new net: C12.2, U4.3 (CH1)
- new net: TP14.1, U4.14 (DOUT), XIAO1.9
- new net: C10.2, U4.20 (REF)
- new net: IC1.9, TP13.1, XIAO1.0
- new net -4.5V: C2.2, C4.2, C6.1, C8.1, IC1.4 (VSS), R2.2, TP2.1, U1.4 (V-), U5.4 (V-), Vbat1.2 (-)
- no-connect marks 23 -> 11
Other:
- note added: "<-- Break in Ground Plane Below this Output"
- note added: "Analog"
- note added: "MISO"
- note added: "MOSI"
- note added: "Microcontroller (QT PY ESP32-S3)"
- note added: "Rx"
- note added: "SCK"
- note added: "SCL"
- note added: "SDA"
- note added: "Tx"
- note removed: "Microcontroller (ESP32-S3)"
- note removed: "OLED display"
- note removed: "Voltage Regulator 5V Output"
