File: Kicad/ECE 412.kicad_pcb (KiCad board)
At the start: 2 copper layers, 53.4 x 65.1 mm, 20 parts, among them J1 Faraday Cup IN, J2 3.3V, U2 3405, U4 LMC662, U5 MAX1032BEUG_

Commit message: Add files via upload
Parts:
- removed J1: Faraday Cup IN, Connector_PinHeader_2.54mm:PinHeader_1x01_P2.54mm_Vertical
- removed J2: 3.3V, Connector_PinHeader_2.54mm:PinHeader_1x02_P2.54mm_Vertical
- removed TP1, TP3, TP4: TestPoint, TestPoint:TestPoint_THTPad_D2.0mm_Drill1.0mm
- added A1: Adafruit_Feather_HUZZAH32_ESP32, Module:Adafruit_Feather, F.Cu at (139.4, 66.6)
- added C1: 10uF, Capacitor_THT:C_Radial_D6.3mm_H5.0mm_P2.50mm, F.Cu at (127.2, 64.6)
- added C2: 0.1uF, Capacitor_THT:C_Radial_D6.3mm_H5.0mm_P2.50mm, F.Cu at (127.2, 71.6)
- added TP10: ADC DIN, TestPoint:TestPoint_THTPad_D2.0mm_Drill1.0mm, F.Cu at (188.8, 110.5)
- added TP12: ADC Dout, TestPoint:TestPoint_THTPad_D2.0mm_Drill1.0mm, F.Cu at (189.1, 101.5)
- added TP5: 470k switch, TestPoint:TestPoint_THTPad_D2.0mm_Drill1.0mm, F.Cu at (177.8, 48.8)
- added TP6: 150k switch, TestPoint:TestPoint_THTPad_D2.0mm_Drill1.0mm, F.Cu at (189.1, 92.0)
- added TP7: 40k switch, TestPoint:TestPoint_THTPad_D2.0mm_Drill1.0mm, F.Cu at (166.0, 48.8)
- added TP9: ADC SCLK, TestPoint:TestPoint_THTPad_D2.0mm_Drill1.0mm, F.Cu at (189.6, 118.0)
- added U1: LM7805_TO220, Package_TO_SOT_THT:TO-220-3_Vertical, F.Cu at (118.9, 63.6)
- C3: value 10uF -> 0.1uF; footprint Capacitor_THT:CP_Radial_D5.0mm_P2.00mm -> Capacitor_THT:C_Radial_D6.3mm_H5.0mm_P2.50mm
- C4: value 10uF -> 1uF; footprint Capacitor_THT:CP_Radial_D5.0mm_P2.00mm -> Capacitor_THT:C_Radial_D6.3mm_H5.0mm_P2.50mm
- C5: footprint Capacitor_THT:CP_Radial_Tantal_D5.0mm_P5.00mm -> Capacitor_THT:C_Radial_D10.0mm_H12.5mm_P5.00mm
- TP2: value TestPoint -> 5V
- U2: value 3405 -> ADG441BN; footprint 3405_Huzzah:MODULE_3405 -> ADG441BN:DIP254P762X533-16P
- U4: footprint LMC662AIMX_NOPB:SOIC127P599X175-8N -> Package_DIP:DIP-8_W7.62mm
- moved R4 86.9 mm to (88.6, 107.4), turned to 90 degrees
- moved R1 80.2 mm to (98.7, 68.7)
- moved C3 76.1 mm to (114.7, 100.8), turned to 0 degrees
- moved R2 74.2 mm to (88.5, 63.0), turned to 0 degrees
- moved Vbat1 73.6 mm to (109.7, 65.0), turned to 180 degrees
- moved R5 69.6 mm to (95.9, 98.5), turned to -90 degrees
- moved TP2 67.5 mm to (163.0, 120.0)
- moved R6 60.8 mm to (102.7, 98.5), turned to -90 degrees
- moved U4 58.5 mm to (89.4, 81.2), turned to 90 degrees
- moved C5 56.2 mm to (88.3, 91.0), turned to -90 degrees
- moved C4 53.7 mm to (122.5, 106.8), turned to 180 degrees
- moved R7 52.8 mm to (109.2, 98.5), turned to -90 degrees
- moved U5 51.4 mm to (129.6, 102.3), turned to 90 degrees
- moved R3 48.9 mm to (88.2, 86.4), turned to 180 degrees
- moved U2 42.8 mm to (123.0, 82.9), turned to 90 degrees
Connections:
- C3 pad 1: Net-(U4-V+) -> GND
- C3 pad 2: GND -> Net-(U5-REF)
- R1 pad 1: Net-(U4-V+) -> /9V
- R5 pad 1: Net-(U4-OUTB) -> Net-(U2-D3)
- R6 pad 1: Net-(U4-OUTB) -> Net-(U2-D2)
- R7 pad 1: Net-(U4-OUTB) -> Net-(U2-D1)
- TP2 pad 1: Net-(U4-OUTA) -> /5V
- U2 pad 1: Net-(U2-IO21) -> Net-(A1-A9/IO33)
- U2 pad 10: unconnected-(U2-A2/IO34-Pad10) -> Net-(U2-D3)
- U2 pad 11: unconnected-(U2-A1_DAC1-Pad11) -> Net-(U2-S1)
- U2 pad 13: GND -> /9V
- U2 pad 14: unconnected-(U2-NC-Pad14) -> Net-(U2-S1)
- U2 pad 15: /3.3V -> Net-(U2-D2)
- U2 pad 16: unconnected-(U2-RST-Pad16) -> Net-(A1-A7/IO32)
- U2 pad 2: Net-(DS1-D/~{C}) -> Net-(U2-D1)
- U2 pad 3: Net-(DS1-~{RES}) -> Net-(U2-S1)
- U2 pad 4: Net-(U2-MISO/IO19) -> GND
- U2 pad 5: Net-(DS1-D5) -> GND
- U2 pad 6: Net-(DS1-D4) -> unconnected-(U2-S4-Pad6)
- U2 pad 8: unconnected-(U2-A4/IO36-Pad8) -> GND
- U2 pad 9: unconnected-(U2-A3/IO39-Pad9) -> Net-(A1-A6/IO14)
- U4 pad 7: Net-(U4-OUTB) -> Net-(U2-S1)
- U4 pad 8: Net-(U4-V+) -> /9V
- U5 pad 1: /3.3V -> /5V
- U5 pad 10: Net-(U2-IO21) -> Net-(A1-I34/A2)
- U5 pad 11: Net-(DS1-D5) -> Net-(A1-MOSI/IO18)
- U5 pad 13: Net-(DS1-D4) -> Net-(A1-SCK/IO5)
- U5 pad 14: Net-(U2-MISO/IO19) -> Net-(A1-MISO/IO19)
- U5 pad 15: unconnected-(U5-DGND0-Pad15) -> GND
- U5 pad 16: unconnected-(U5-DGND-Pad16) -> GND
- U5 pad 17: unconnected-(U5-DVDD0-Pad17) -> /3.3V
- U5 pad 18: unconnected-(U5-DVDD-Pad18) -> /3.3V
- U5 pad 2: Net-(U4-OUTB) -> Net-(U2-S1)
- U5 pad 20: /3.3V -> Net-(U5-REF)
- U5 pad 21: unconnected-(U5-AGND3-Pad21) -> GND
- U5 pad 22: unconnected-(U5-AVDD2-Pad22) -> /5V
- U5 pad 23: unconnected-(U5-AGND2-Pad23) -> GND
- U5 pad 3: unconnected-(U5-CH1-Pad3) -> GND
- U5 pad 4: unconnected-(U5-CH2-Pad4) -> GND
- U5 pad 5: unconnected-(U5-CH3-Pad5) -> GND
- Vbat1 pad 1: Net-(U4-V+) -> /9V
Routing:
- net /5V: track 0.00 -> 150.6 mm, vias 0 -> 3
- net Net-(U2-S1): track 0.00 -> 98.4 mm
- net Net-(U4-OUTB): track 72.4 -> 0.00 mm
- net Net-(A1-A9/IO33): track 0.00 -> 71.0 mm
- net /9V: track 0.00 -> 66.5 mm, vias 0 -> 1
- net Net-(A1-A7/IO32): track 0.00 -> 63.8 mm
- net Net-(U2-MISO/IO19): track 56.6 -> 0.00 mm, vias 1 -> 0
- net Net-(U2-D2): track 0.00 -> 52.0 mm
- net Net-(U4-V+): track 51.7 -> 0.00 mm, vias 1 -> 0
- net Net-(A1-A6/IO14): track 0.00 -> 43.6 mm
- net Net-(U2-IO21): track 40.2 -> 0.00 mm
- net Net-(A1-I34/A2): track 0.00 -> 37.3 mm
- net /Faraday Cup: track 36.5 -> 0.00 mm
- net Net-(DS1-D5): track 34.6 -> 0.00 mm, vias 1 -> 0
- net Net-(U2-D3): track 0.00 -> 33.4 mm
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Other:
- board size 53.4 x 65.1 mm -> 91.4 x 52.5 mm

Commit message: Add files via upload
Parts:
- removed U2: ADG441BN, ADG441BN:DIP254P762X533-16P
- added C10: 0.1uF, Capacitor_SMD:C_0805_2012Metric_Pad1.18x1.45mm_HandSolder, F.Cu at (121.0, 94.3)
- added C11: 0.1uF, Capacitor_SMD:C_0805_2012Metric_Pad1.18x1.45mm_HandSolder, F.Cu at (132.5, 90.8)
- added C12: 100pF, Capacitor_SMD:C_0805_2012Metric_Pad1.18x1.45mm_HandSolder, F.Cu at (122.3, 105.1)
- added C13: 0.1uF, Capacitor_SMD:C_0805_2012Metric_Pad1.18x1.45mm_HandSolder, F.Cu at (123.5, 108.7)
- added C14: 0.1uF, Capacitor_SMD:C_0805_2012Metric_Pad1.18x1.45mm_HandSolder, F.Cu at (128.1, 108.7)
- added C15: 0.1uF, Capacitor_SMD:C_0805_2012Metric_Pad1.18x1.45mm_HandSolder, F.Cu at (128.8, 105.0)
- added C16: 10uF, Capacitor_SMD:C_0805_2012Metric_Pad1.18x1.45mm_HandSolder, F.Cu at (114.0, 65.0)
- added C17: 0.1uF, Capacitor_SMD:C_0805_2012Metric_Pad1.18x1.45mm_HandSolder, F.Cu at (113.9, 61.6)
- added C18: 10uF, Capacitor_SMD:C_0805_2012Metric_Pad1.18x1.45mm_HandSolder, F.Cu at (88.1, 63.2)
- added C19: 0.1uF, Capacitor_SMD:C_0805_2012Metric_Pad1.18x1.45mm_HandSolder, F.Cu at (93.2, 63.2)
- added C6: 10uF, Capacitor_SMD:C_0805_2012Metric_Pad1.18x1.45mm_HandSolder, F.Cu at (120.9, 97.6)
- added C7: 0.1uF, Capacitor_SMD:C_0805_2012Metric_Pad1.18x1.45mm_HandSolder, F.Cu at (120.9, 101.0)
- added C8: 0.1uF, Capacitor_SMD:C_0805_2012Metric_Pad1.18x1.45mm_HandSolder, F.Cu at (129.8, 90.7)
- added C9: 1uF, Capacitor_SMD:C_0805_2012Metric_Pad1.18x1.45mm_HandSolder, F.Cu at (135.2, 90.8)
- added IC1: ADG412, ADG412:TSSOP16, F.Cu at (110.1, 77.8)
- added REF**: MountingHole_3.2mm_M3, MountingHole:MountingHole_3.2mm_M3, F.Cu at (166.2, 108.0)
- added REF**: MountingHole_3.2mm_M3, MountingHole:MountingHole_3.2mm_M3, F.Cu at (82.0, 108.0)
- added REF**: MountingHole_3.2mm_M3, MountingHole:MountingHole_3.2mm_M3, F.Cu at (166.0, 64.0)
- added REF**: MountingHole_3.2mm_M3, MountingHole:MountingHole_3.2mm_M3, F.Cu at (81.9, 63.5)
- added REF**: MountingHole_4.3mm_M4_DIN965_Pad, MountingHole:MountingHole_4.3mm_M4_DIN965_Pad, F.Cu at (73.6, 85.8)
- added TP1: 4.5V, TestPoint:TestPoint_THTPad_D2.0mm_Drill1.0mm, F.Cu at (80.0, 99.0)
- added TP11: ADC CS, TestPoint:TestPoint_THTPad_D2.0mm_Drill1.0mm, F.Cu at (166.0, 73.0)
- added TP3: Vout1, TestPoint:TestPoint_THTPad_D2.0mm_Drill1.0mm, F.Cu at (80.0, 76.2)
- added TP4: Vout2, TestPoint:TestPoint_THTPad_D2.0mm_Drill1.0mm, F.Cu at (80.0, 69.8)
- added TP8: ADC Vref, TestPoint:TestPoint_THTPad_D2.0mm_Drill1.0mm, F.Cu at (123.4, 80.0)
- C1, C2, C4: footprint Capacitor_THT:C_Radial_D6.3mm_H5.0mm_P2.50mm -> Capacitor_SMD:C_0805_2012Metric_Pad1.18x1.45mm_HandSolder
- C3: value 0.1uF -> 1uF; footprint Capacitor_THT:C_Radial_D6.3mm_H5.0mm_P2.50mm -> Capacitor_SMD:C_0805_2012Metric_Pad1.18x1.45mm_HandSolder
- TP5: value 470k switch -> 470k
- TP6: value 150k switch -> 150k
- TP7: value 40k switch -> 40k
- moved TP5 92.3 mm to (105.0, 105.5)
- moved TP6 90.1 mm to (100.0, 105.5)
- moved TP7 80.1 mm to (109.5, 105.5)
- moved TP2 50.6 mm to (114.5, 105.5)
- moved TP9 43.4 mm to (166.0, 81.5), turned to 90 degrees
- moved TP10 30.6 mm to (166.0, 90.0), turned to 90 degrees
- moved TP12 23.2 mm to (166.0, 99.0), turned to 90 degrees
- moved C4 16.4 mm to (126.3, 90.8), turned to 90 degrees
- moved C3 13.4 mm to (123.7, 90.8), turned to -90 degrees
- moved Vbat1 12.3 mm to (121.6, 61.8), turned to 0 degrees
- moved R5 11.1 mm to (101.5, 89.0)
- moved R4 10.8 mm to (94.6, 98.4), turned to 180 degrees
- moved R6 10.7 mm to (107.7, 89.0)
- moved R7 10.6 mm to (113.8, 89.0)
- moved C2 9.95 mm to (133.0, 63.5)
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Connections:
- U5 pad 3: GND -> Net-(U5-CH1)
- U5 pad 4: GND -> Net-(U5-CH2)
- U5 pad 5: GND -> Net-(U5-CH3)
Routing:
- net Net-(A1-A6/IO14): track 43.6 -> 98.1 mm, vias 0 -> 1
- net Net-(A1-A7/IO32): track 63.8 -> 105.4 mm, vias 0 -> 1
- net Net-(IC1-Pad15): track 52.0 -> 15.5 mm
- net Net-(A1-A9/IO33): track 71.0 -> 106.8 mm, vias 0 -> 2
- net /4.5V: track 32.7 -> 65.2 mm
- net Net-(A1-SCK/IO5): track 9.95 -> 40.0 mm, vias 0 -> 1
- net Net-(A1-MISO/IO19): track 9.61 -> 38.0 mm
- net /5V: track 150.6 -> 127.4 mm, vias 3 -> 0
- net Net-(U4-OUTB): track 98.4 -> 75.7 mm, vias 0 -> 2
- net GND: track 0.00 -> 21.1 mm, vias 0 -> 13
- net Net-(A1-MOSI/IO18): track 22.3 -> 40.0 mm
- net Net-(A1-I34/A2): track 37.3 -> 52.8 mm
- net Net-(IC1-Pad10): track 33.4 -> 18.9 mm, vias 0 -> 1
- net Net-(IC1-Pad2): track 23.4 -> 10.5 mm
- net Net-(U4-NEGB): track 57.9 -> 46.8 mm
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Other:
- board size 91.4 x 52.5 mm -> 102.8 x 52.6 mm
- board text added: "Switches"
- board text added: "Team 3: COATL Aircraft Sensor"

Commit message: Add files via upload
Parts:
- IC1: footprint ADG412:TSSOP16 -> ADG412:SOIC16N
- moved C10 1.48 mm to (119.5, 94.2)
- moved C6 1.48 mm to (119.5, 97.5)
- moved C7 1.48 mm to (119.5, 100.8)
- moved R5 1.30 mm to (100.2, 89.1)
- moved R6 1.30 mm to (106.4, 89.1)
- moved R7 1.30 mm to (112.5, 89.1)
- moved IC1 1.09 mm to (109.5, 78.7), turned to 0 degrees
Routing:
- net GND: track 21.1 -> 41.5 mm, vias 13 -> 17
- net Net-(A1-MOSI/IO18): track 40.0 -> 48.8 mm, vias 0 -> 1
- net Net-(A1-A9/IO33): track 106.8 -> 115.4 mm, vias 2 -> 1
- net /5V: track 127.4 -> 134.8 mm, vias 0 -> 1
- net Net-(IC1-Pad10): track 18.9 -> 26.0 mm
- net Net-(IC1-Pad15): track 15.5 -> 20.4 mm
- net Net-(A1-I34/A2): track 52.8 -> 57.3 mm, vias 0 -> 1
- net Net-(A1-A7/IO32): track 105.4 -> 109.2 mm
- net Net-(U4-OUTB): track 75.7 -> 79.0 mm, vias 2 -> 3
- net Net-(IC1-Pad2): track 10.5 -> 12.7 mm
- net /9V: track 56.9 -> 57.8 mm
- net Net-(A1-A6/IO14): track 98.1 -> 97.4 mm
- net Net-(A1-MISO/IO19): track 38.0 -> 38.7 mm
- net /3.3V: track 39.7 -> 39.8 mm, vias 0 -> 1
Other:
- board size 102.8 x 52.6 mm -> 102.8 x 52.5 mm

Commit message: Add files via upload
Parts:
- C1: value 10uF -> 1uF; footprint Capacitor_SMD:C_0805_2012Metric_Pad1.18x1.45mm_HandSolder -> Capacitor_SMD:C_1206_3216Metric_Pad1.33x1.80mm_HandSolder
- C10, C11, C12, C13, C14, C15, C16, C17, C18, C19, C2, C3, C4, C6, C7, C8, C9: footprint Capacitor_SMD:C_0805_2012Metric_Pad1.18x1.45mm_HandSolder -> Capacitor_SMD:C_1206_3216Metric_Pad1.33x1.80mm_HandSolder
- R1, R2, R4, R5, R6, R7: footprint XIAO_:R_Axial_DIN0207_L6.3mm_D2.5mm_P10.16mm_Horizontal_2.54_pad -> Resistor_SMD:R_0805_2012Metric_Pad1.20x1.40mm_HandSolder
- U1: value LM7805_TO220 -> LM7805
- moved R7 7.05 mm to (109.3, 95.4)
- moved R6 6.75 mm to (103.9, 95.4)
- moved C9 6.73 mm to (133.6, 84.3), turned to 180 degrees
- moved R5 6.51 mm to (98.5, 95.4)
- moved R1 5.95 mm to (102.0, 63.8), turned to 90 degrees
- moved C17 5.68 mm to (108.5, 63.5), turned to -90 degrees
- moved C18 5.59 mm to (93.7, 63.3)
- moved C19 5.07 mm to (88.1, 63.3)
- moved C6 5.02 mm to (115.3, 100.4), turned to -90 degrees
- moved IC1 4.09 mm to (106.2, 81.1)
- moved C14 3.57 mm to (131.6, 109.4)
- moved C13 3.39 mm to (120.1, 109.4)
- moved TP2 3.27 mm to (111.2, 105.6)
- moved Vbat1 2.82 mm to (118.8, 61.8)
- moved U1 2.79 mm to (123.7, 63.4), turned to 0 degrees
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Routing:
- net Net-(A1-MOSI/IO18): track 48.8 -> 40.3 mm, vias 1 -> 0
- net /4.5V: track 65.2 -> 56.8 mm, vias 0 -> 2
- net Net-(A1-A9/IO33): track 115.4 -> 109.2 mm
- net Net-(U4-NEGB): track 47.2 -> 41.4 mm
- net Net-(IC1-Pad10): track 26.0 -> 21.0 mm, vias 1 -> 2
- net Net-(A1-I34/A2): track 57.3 -> 52.9 mm, vias 1 -> 0
- net Net-(U4-OUTB): track 79.0 -> 82.6 mm
- net Net-(A1-A7/IO32): track 109.2 -> 106.4 mm, vias 1 -> 2
- net /9V: track 57.8 -> 59.9 mm, vias 1 -> 0
- net Net-(U5-CH2): track 8.49 -> 10.4 mm
- net Net-(U5-CH1): track 8.60 -> 10.5 mm
- net Net-(IC1-Pad15): track 20.4 -> 18.7 mm
- net /3.3V: track 39.8 -> 38.3 mm, vias 1 -> 0
- net Net-(U4-OUTA): track 26.9 -> 28.3 mm
- net Net-(U5-CH3): track 4.87 -> 6.23 mm
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Other:
- board size 102.8 x 52.5 mm -> 102.8 x 52.4 mm
- board text added: "Switch Outputs"
- board text removed: "Switches"

Commit message: Add files via upload
Routing:
- net GND: vias 22 -> 21
Changed lines of the file:
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@@
 	(title_block
 		(title "Team 3 - COATL Aircraft PCB")
-		(date "2025-04-06")
+		(date "2025-04-07")
 		(rev "C")
 		(company "Annika Boyd, Eisa Alsharifi, Felix Moss, Nathan Truong")
@@
 	)
 	(via
-		(at 94 89)
-		(size 0.6)
-		(drill 0.3)
-		(layers "F.Cu" "B.Cu")
-		(free yes)
-		(net 1)
-	)
-	(via
-		(at 94.635 84.895)
+		(at 94.01 84.695)
 		(size 0.6)
 		(drill 0.3)

Commit message: Add files via upload
Parts:
- added G***: LOGO, LOGO, F.Cu at (89.6, 105.3)
- moved C17 20.6 mm to (88.0, 63.3), turned to 90 degrees
- moved REF** 9.34 mm to (64.3, 85.6)
- moved Vbat1 6.68 mm to (112.1, 61.9)
- moved C19 5.30 mm to (93.4, 63.2)
- moved C18 5.08 mm to (98.8, 63.2)
- moved R2 5.08 mm to (103.4, 63.7)
- moved R1 5.08 mm to (107.1, 63.7), turned to -90 degrees
- moved C16 3.53 mm to (117.5, 63.5)
- moved TP12 3.22 mm to (166.3, 95.8)
- moved TP10 2.52 mm to (166.3, 87.5)
- moved TP11 2.48 mm to (166.0, 70.5)
- moved TP9 2.36 mm to (166.2, 79.1)
- moved TP5 0.70 mm to (102.2, 104.9)
- moved TP6 0.70 mm to (97.2, 104.9)
- moved TP7 0.70 mm to (106.7, 104.9)
Routing:
- net Net-(A1-A6/IO14): track 98.0 -> 89.0 mm
- net Net-(A1-A7/IO32): track 106.4 -> 100.1 mm
- net Net-(A1-A9/IO33): track 109.2 -> 104.0 mm
- net /4.5V: track 56.8 -> 61.5 mm
- net /9V: track 59.9 -> 63.6 mm
- net Net-(A1-I34/A2): track 52.9 -> 55.4 mm
- net Net-(A1-MOSI/IO18): track 40.3 -> 41.6 mm
- net Net-(A1-SCK/IO5): track 40.0 -> 41.2 mm
- net Net-(A1-MISO/IO19): track 37.9 -> 38.9 mm
Other:
- board size 102.8 x 52.4 mm -> 112.7 x 52.4 mm

Commit message: Add files via upload
Parts:
- removed A1: Adafruit_Feather_HUZZAH32_ESP32, Module:Adafruit_Feather
- removed TP10: ADC DIN, TestPoint:TestPoint_THTPad_D2.0mm_Drill1.0mm
- added C20: 0.1uF, Capacitor_SMD:C_1206_3216Metric_Pad1.33x1.80mm_HandSolder, F.Cu at (138.2, 90.6)
- added C21: 0.1uF, Capacitor_SMD:C_1206_3216Metric_Pad1.33x1.80mm_HandSolder, F.Cu at (117.9, 88.5)
- added TP13: 40k, TestPoint:TestPoint_THTPad_D2.0mm_Drill1.0mm, F.Cu at (97.1, 105.6)
- added TP14: ADC Dout, TestPoint:TestPoint_THTPad_D2.0mm_Drill1.0mm, F.Cu at (152.7, 108.1)
- added XIAO1: ~, XIAO_:XIAO_QTpy, F.Cu at (169.4, 87.5)
- C1: value 1uF -> 100p; footprint Capacitor_SMD:C_1206_3216Metric_Pad1.33x1.80mm_HandSolder -> Capacitor_THT:C_Radial_D10.0mm_H12.5mm_P5.00mm
- C10, C11, C19: value 0.1uF -> 1uF
- C12: value 100pF -> 0.1uF
- C18, C6: value 10uF -> 0.1uF
- C2: value 0.1uF -> 10uF
- C3, C4: value 1uF -> 10uF
- C5: value 100p -> 0.1uF; footprint Capacitor_THT:C_Radial_D10.0mm_H12.5mm_P5.00mm -> Capacitor_SMD:C_1206_3216Metric_Pad1.33x1.80mm_HandSolder
- C9: value 1uF -> 100pF
- R5: value 40k -> 470k
- R7: value 470k -> 40k
- TP11: value ADC CS -> 470k
- TP12: value ADC Dout -> 150k
- TP2: value 5V -> -4.5V
- TP4: value Vout2 -> 0V
- TP5: value 470k -> Vout2
- TP6: value 150k -> ADC Vref
- TP7: value 40k -> ADC SCLK
- TP8: value ADC Vref -> ADC DIN
- TP9: value ADC SCLK -> ADC CS
- U1: value LM7805 -> LMC662; footprint Package_TO_SOT_THT:TO-220-3_Vertical -> Package_DIP:DIP-8_W7.62mm
- U4: value LMC662 -> MAX1032BEUG_; footprint Package_DIP:DIP-8_W7.62mm -> MAX1032BEUGT:SOP65P640X110-24N
- U5: value MAX1032BEUG_ -> BUF634AxD; footprint MAX1032BEUGT:SOP65P640X110-24N -> Package_SO:SOIC-8_3.9x4.9mm_P1.27mm
- moved TP11 69.1 mm to (106.5, 105.7), turned to 0 degrees
- moved TP12 65.3 mm to (101.7, 105.6), turned to 0 degrees
- moved C1 56.8 mm to (81.4, 90.3), turned to 180 degrees
- moved C17 49.1 mm to (124.9, 95.7), turned to 180 degrees
- moved U4 48.9 mm to (132.3, 98.0)
- moved C19 48.1 mm to (136.4, 84.8)
- moved U1 46.2 mm to (81.3, 81.8), turned to 90 degrees
- moved TP8 46.0 mm to (159.8, 108.1)
- moved TP1 45.1 mm to (109.6, 65.0)
- moved C18 45.0 mm to (134.5, 90.7), turned to -90 degrees
- moved TP5 42.5 mm to (88.8, 64.5)
- moved TP2 41.2 mm to (104.1, 65.0)
- moved Vbat1 39.6 mm to (151.4, 66.2), turned to 180 degrees
- moved R2 39.5 mm to (142.9, 63.2), turned to 0 degrees
- moved TP6 39.4 mm to (129.1, 81.6)
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Connections:
- C1 pad 1: /5V -> Net-(U1-OUTA)
- C10 pad 1: /5V -> GND
- C10 pad 2: GND -> Net-(U4-REF)
- C11 pad 1: GND -> Net-(U4-REFCAP)
- C11 pad 2: /3.3V -> GND
- C12 pad 2: Net-(U4-OUTB) -> Net-(U4-CH1)
- C13 pad 2: Net-(U5-CH1) -> Net-(U4-CH2)
- C14 pad 2: Net-(U5-CH2) -> Net-(U4-CH3)
- C15 pad 1: GND -> /4.5V
- C15 pad 2: Net-(U5-CH3) -> GND
- C16 pad 1: /9V -> /4.5V
- C17 pad 1: /9V -> /4.5V
- C18 pad 1: /4.5V -> GND
- C18 pad 2: GND -> /3.3V
- C19 pad 1: /4.5V -> /3.3V
- C2 pad 1: /5V -> /4.5V
- C2 pad 2: GND -> /-4.5V
- C3 pad 1: GND -> /4.5V
- C3 pad 2: Net-(U5-REF) -> GND
- C4 pad 1: Net-(U5-REFCAP) -> GND
- C4 pad 2: GND -> /-4.5V
- C5 pad 1: Net-(U4-OUTA) -> /4.5V
- C6 pad 1: /5V -> /-4.5V
- C7 pad 1: /5V -> /4.5V
- C8 pad 1: GND -> /-4.5V
- C8 pad 2: /3.3V -> GND
- C9 pad 1: /3.3V -> GND
- C9 pad 2: GND -> Net-(U1-OUTB)
- IC1 pad 1: Net-(A1-A9/IO33) -> Net-(IC1-Pad1)
- IC1 pad 11: Net-(U4-OUTB) -> Net-(U1-OUTB)
- IC1 pad 12: /5V -> /3.3V
- IC1 pad 13: /9V -> /4.5V
- IC1 pad 14: Net-(U4-OUTB) -> Net-(U1-OUTB)
- IC1 pad 16: Net-(A1-A7/IO32) -> Net-(IC1-Pad16)
- IC1 pad 3: Net-(U4-OUTB) -> Net-(U1-OUTB)
- IC1 pad 4: GND -> /-4.5V
- IC1 pad 9: Net-(A1-A6/IO14) -> Net-(IC1-Pad9)
- R1 pad 1: /9V -> /4.5V
- R1 pad 2: /4.5V -> Net-(U5-V_{IN})
- R2 pad 1: /4.5V -> Net-(U5-V_{IN})
- R2 pad 2: GND -> /-4.5V
- R3 pad 1: Net-(U4-OUTA) -> Net-(U1-OUTA)
- R4 pad 1: Net-(U4-NEGB) -> Net-(U1-NEGB)
- R4 pad 2: Net-(U4-OUTA) -> Net-(U1-OUTA)
- R5 pad 1: Net-(IC1-Pad10) -> Net-(IC1-Pad2)
- R5 pad 2: Net-(U4-NEGB) -> Net-(U1-NEGB)
- R6 pad 2: Net-(U4-NEGB) -> Net-(U1-NEGB)
- R7 pad 1: Net-(IC1-Pad2) -> Net-(IC1-Pad10)
- R7 pad 2: Net-(U4-NEGB) -> Net-(U1-NEGB)
- TP11 pad 1: Net-(A1-I34/A2) -> Net-(IC1-Pad1)
- TP12 pad 1: Net-(A1-MISO/IO19) -> Net-(IC1-Pad16)
- TP2 pad 1: /5V -> /-4.5V
- TP3 pad 1: Net-(U4-OUTA) -> Net-(U1-OUTA)
- TP4 pad 1: Net-(U4-OUTB) -> GND
- TP5 pad 1: Net-(A1-A9/IO33) -> Net-(U1-OUTB)
- TP6 pad 1: Net-(A1-A7/IO32) -> Net-(U4-REFCAP)
- TP7 pad 1: Net-(A1-A6/IO14) -> Net-(U4-SCLK)
- TP8 pad 1: Net-(U5-REFCAP) -> Net-(U4-DIN)
- TP9 pad 1: Net-(A1-SCK/IO5) -> Net-(U4-~{CS})
- U1 pad 1: /9V -> Net-(U1-OUTA)
- U1 pad 3: /5V -> GND
- U4 pad 1: Net-(U4-OUTA) -> /4.5V
- U4 pad 3: /4.5V -> Net-(U4-CH1)
- U4 pad 4: GND -> Net-(U4-CH2)
- U4 pad 5: /4.5V -> Net-(U4-CH3)
- U4 pad 6: Net-(U4-NEGB) -> unconnected-(U4-CH4-Pad6)
- U4 pad 7: Net-(U4-OUTB) -> unconnected-(U4-CH5-Pad7)
- U4 pad 8: /9V -> unconnected-(U4-CH6-Pad8)
- U5 pad 1: /5V -> unconnected-(U5-BW-Pad1)
- U5 pad 2: Net-(U4-OUTB) -> unconnected-(U5-NC-Pad2)
- U5 pad 3: Net-(U5-CH1) -> Net-(U5-V_{IN})
- U5 pad 4: Net-(U5-CH2) -> /-4.5V
- U5 pad 5: Net-(U5-CH3) -> unconnected-(U5-NC-Pad5)
- U5 pad 6: unconnected-(U5-CH4-Pad6) -> GND
- U5 pad 7: unconnected-(U5-CH5-Pad7) -> /4.5V
- Vbat1 pad 1: /9V -> /4.5V
- Vbat1 pad 2: GND -> /-4.5V
Routing:
- net /5V: track 135.1 -> 0.00 mm
- net /4.5V: track 61.5 -> 193.0 mm, vias 2 -> 0
- net Net-(A1-A9/IO33): track 104.0 -> 0.00 mm, vias 1 -> 0
- net Net-(IC1-Pad1): track 0.00 -> 101.1 mm, vias 0 -> 1
- net Net-(A1-A7/IO32): track 100.1 -> 0.00 mm, vias 2 -> 0
- net /-4.5V: track 0.00 -> 98.1 mm, vias 0 -> 2
- net Net-(IC1-Pad9): track 0.00 -> 97.5 mm, vias 0 -> 2
- net Net-(IC1-Pad16): track 0.00 -> 93.6 mm, vias 0 -> 2
- net Net-(U1-OUTB): track 0.00 -> 90.4 mm
- net Net-(A1-A6/IO14): track 89.0 -> 0.00 mm, vias 1 -> 0
- net Net-(U4-OUTB): track 82.6 -> 0.00 mm, vias 3 -> 0
- net /9V: track 63.6 -> 0.00 mm
- net Net-(U4-~{CS}): track 0.00 -> 60.1 mm, vias 0 -> 1
- net Net-(A1-I34/A2): track 55.4 -> 0.00 mm
- net Net-(U1-OUTA): track 0.00 -> 53.5 mm
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
Commit message: Add files via upload
Parts:
- moved C21 2.66 mm to (115.2, 88.9)
